Commit message: added robot_launch file

File: urdf/my_robot.xacro (robot description, xacro)
@@ -149,5 +149,5 @@
     <mu2 value = "0.001"/>
   </gazebo>
-  <link name="lidar">
+  <link name="laser_frame">
     <inertial>
       <origin xyz="-0.002361 -1.4968E-05 0.019299" rpy="0 0 0" />
@@ -183,5 +183,5 @@
   <gazebo reference="lidar">
         <material>Gazebo/Black</material>
-        <sensor name="laser" type="ray">
+        <sensor name="laser_frame" type="ray">
             <pose> 0 0 0 0 0 0 </pose>
             <visualize>true</visualize>
@@ -205,5 +205,5 @@
                 </ros>
                 <output_type>sensor_msgs/LaserScan</output_type>
-                <frame_name>lidar</frame_name>
+                <frame_name>laser_frame</frame_name>
             </plugin>
         </sensor>
